File: PiWing/PiWing.brd (EAGLE design)
At the start: 65.6 x 30.1 mm, 8 parts

Commit message: Updated PiWing
Routing:
- net 3V: track 85.3 -> 81.9 mm
Changed lines of the file:
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@@
 <grid distance="50" unitdist="mil" unit="mil" style="lines" multiple="1" display="no" altdistance="5" altunitdist="mil" altunit="mil"/>
 <layers>
-<layer number="1" name="Top" color="4" fill="1" visible="no" active="yes"/>
-<layer number="16" name="Bottom" color="1" fill="1" visible="no" active="yes"/>
+<layer number="1" name="Top" color="4" fill="1" visible="yes" active="yes"/>
+<layer number="16" name="Bottom" color="1" fill="1" visible="yes" active="yes"/>
 <layer number="17" name="Pads" color="2" fill="1" visible="yes" active="yes"/>
 <layer number="18" name="Vias" color="2" fill="1" visible="yes" active="yes"/>
@@
 <layer number="23" name="tOrigins" color="15" fill="1" visible="yes" active="yes"/>
 <layer number="24" name="bOrigins" color="15" fill="1" visible="no" active="yes"/>
-<layer number="25" name="tNames" color="7" fill="1" visible="yes" active="yes"/>
+<layer number="25" name="tNames" color="7" fill="1" visible="no" active="yes"/>
 <layer number="26" name="bNames" color="7" fill="1" visible="yes" active="yes"/>
 <layer number="27" name="tValues" color="7" fill="1" visible="yes" active="yes"/>
@@
 <text x="31.75" y="27.94" size="0.762" layer="25" align="bottom-center">TX</text>
 <text x="34.29" y="27.94" size="0.762" layer="25" align="bottom-center">RX</text>
-<text x="24.13" y="19.304" size="0.762" layer="25" align="bottom-center">SDA</text>
-<text x="26.67" y="19.304" size="0.762" layer="25" align="bottom-center">SCL</text>
+<text x="26.67" y="19.304" size="0.762" layer="25" align="bottom-center">SDA</text>
+<text x="29.21" y="19.304" size="0.762" layer="25" align="bottom-center">SCL</text>
 <text x="46.99" y="19.304" size="0.762" layer="25" align="bottom-center">MO</text>
 <text x="49.53" y="19.304" size="0.762" layer="25" align="bottom-center">MI</text>
@@
 <text x="69.85" y="21.209" size="0.8128" layer="26" rot="MR180" align="bottom-center">26</text>
 <text x="72.39" y="21.209" size="0.8128" layer="26" rot="MR180" align="bottom-center">GND</text>
-<text x="24.257" y="20.193" size="0.762" layer="26" rot="MR180" align="bottom-center">SDA</text>
-<text x="26.67" y="20.193" size="0.762" layer="26" rot="MR180" align="bottom-center">SCL</text>
+<text x="26.797" y="20.193" size="0.762" layer="26" rot="MR180" align="bottom-center">SDA</text>
+<text x="29.21" y="20.193" size="0.762" layer="26" rot="MR180" align="bottom-center">SCL</text>
 <text x="46.99" y="20.066" size="0.762" layer="26" rot="MR180" align="bottom-center">MO</text>
 <text x="49.53" y="20.066" size="0.762" layer="26" rot="MR180" align="bottom-center">MI</text>
@@
 <wire x1="25.4" y1="30.48" x2="25.4" y2="24.13" width="0.2032" layer="16"/>
 <wire x1="25.4" y1="24.13" x2="24.13" y2="22.86" width="0.2032" layer="16"/>
-<wire x1="76.454" y1="30.988" x2="76.454" y2="20.574" width="0.2032" layer="1"/>
-<wire x1="73.66" y1="17.78" x2="52.07" y2="17.78" width="0.2032" layer="1"/>
 <via x="52.07" y="17.78" extent="1-16" drill="0.35"/>
 <wire x1="52.07" y1="17.78" x2="26.67" y2="17.78" width="0.2032" layer="16"/>
@@
 <wire x1="26.67" y1="17.78" x2="24.13" y2="21.59" width="0.2032" layer="1"/>
 <wire x1="24.13" y1="21.59" x2="24.13" y2="22.86" width="0.2032" layer="1"/>
-<wire x1="76.454" y1="20.574" x2="73.66" y2="17.78" width="0.2032" layer="1"/>
+<wire x1="76.454" y1="30.988" x2="73.5076" y2="28.0416" width="0.1524" layer="1"/>
+<wire x1="73.5076" y1="28.0416" x2="73.5076" y2="24.93706875" width="0.1524" layer="1"/>
+<wire x1="73.5076" y1="24.93706875" x2="72.70053125" y2="24.13" width="0.1524" layer="1"/>
+<wire x1="72.70053125" y1="24.13" x2="58.42" y2="24.13" width="0.1524" layer="1"/>
+<wire x1="58.2676" y1="22.39706875" x2="57.61293125" y2="21.7424" width="0.1524" layer="1"/>
+<wire x1="58.42" y1="24.13" x2="58.2676" y2="23.9776" width="0.1524" layer="1"/>
+<wire x1="56.0324" y1="21.7424" x2="52.07" y2="17.78" width="0.1524" layer="1"/>
+<wire x1="58.2676" y1="23.9776" x2="58.2676" y2="22.39706875" width="0.1524" layer="1"/>
+<wire x1="57.61293125" y1="21.7424" x2="56.0324" y2="21.7424" width="0.1524" layer="1"/>
 </signal>
 <signal name="N$25">
