File: SwitchBoard/Eagle/RelayWing.sch (EAGLE design)
At the start: 30 parts, among them K1 EE2-3TNUH, K2 EE2-3TNUH, K3 EE2-3TNUH, K4 EE2-3TNUH, K5 EE2-3TNUH, U1 ULN2003ANS, U2 ULN2003ANS, U3 MCP23017SS, U4 INA219AID

Commit message: Rev B (start)
First commit for Rev B. See updated Description.
Parts:
- removed I2CHDR: (no value), pinhead:PINHD-2X2
- removed PWR: (no value), led:LEDSMT1206
- added C3: MUR-1220-CAP, home:MUR-1220-CAP
- added JP4, JP5, JP6, JP7: (no value), adafruit:PINHD-1X1CB
- added POWER: HSMQ-C191, DigiKey:HSMQ-C191
- added R2: 330, home:R-US_01005
- RN1: value CTS746X101 -> CTS746X101102JP; device home:CTS746X101 -> home:CTS746X
Connections:
- net N$16 renamed K1A-NO
- net N$17 renamed K2A-NO
- net N$2 renamed K4B-NO
- net N$24 renamed K1-SET
- net N$25 renamed K4B-NC
- net N$26 renamed K2A-CO
- net N$27 renamed K2A-NC
- net N$28 renamed K1A-NC
- net N$29 renamed K1B-NC
- net N$30 renamed K1A-CO
- net N$32 renamed K1B-CO
- net N$33 renamed K2B-CO
- net N$34 renamed K1-RESET
- net N$35 renamed K1B-NO
- net N$36 renamed K2-SET
- net N$37 renamed K2-RESET
- net N$38 renamed K3-SET
- net N$39 renamed K3-RESET
- net N$40 renamed K4A-CO
- net N$42 renamed K4A-N0
- net N$43 renamed K5A-CO
- net N$44 renamed K5A-NO
- net N$45 renamed K5B-NC
- net N$46 renamed K5B-CO
- net N$47 renamed K5B-NO
- net N$49 renamed K4B-CO
- net N$50 renamed K5A-NC
- net N$52 renamed K3A-NO
- net N$53 renamed K3A-NC
- net N$54 renamed K3A-CO
- net N$55 renamed K3B-NO
- net N$56 renamed K3B-NC
- net N$57 renamed K3B-CO
- net N$58 renamed K4-SET
- net N$59 renamed K4-RESET
- net N$60 renamed K5-SET
- net N$72 renamed K2B-NO
- net N$73 renamed K5-RESET
- net N$78 renamed K2B-NC
- net N$79 renamed K4A-NC
- removed net N$18: JP2.1, MS1.!RESET, RESET.S, U3.!RESET
- new net N$31: R2.2, RESET.P
- new net RESET/: C3.C2, JP2.1, MS1.!RESET, RESET.S, RN1.9, U3.!RESET
- net 3V: now also JP4.1, POWER.33; no longer I2CHDR.3, PWR.A
- net GND: now also C3.C1, JP5.1, POWER.11, R2.1; no longer I2CHDR.1, PWR.C, RESET.P
- net SCL: now also JP6.1; no longer I2CHDR.2
- net SDA: now also JP7.1; no longer I2CHDR.4

Commit message: resistor & routing changes
Added LED resistor, resized resisitor to 0603, relocate reset cap.
Parts:
- added R3: 75, home:R-US_R0603
- R2: device home:R-US_01005 -> home:R-US_R0603
Connections:
- net N$62 renamed GPA0
- net N$63 renamed GPB0
- net N$64 renamed GPA1
- net N$65 renamed GPA2
- net N$66 renamed GPB2
- net N$67 renamed GPB1
- net N$68 renamed GPA3
- net N$69 renamed GPB3
- net N$70 renamed GPA4
- net N$71 renamed GPB4
- net N$74 renamed GPA7
- net N$75 renamed GPB5
- net N$76 renamed GPB6
- net N$77 renamed GPB7
- net N$80 renamed GPA5
- net N$81 renamed GPA6
- new net N$2: POWER.33, R3.1
- net 3V: now also R3.2; no longer POWER.33
Changed lines of the file:
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@@
 <part name="JP7" library="adafruit" library_urn="urn:adsk.eagle:library:420" deviceset="PINHD-1X1" device="CB"/>
 <part name="POWER" library="DigiKey" deviceset="HSMQ-C191" device=""/>
-<part name="R2" library="home" deviceset="R-US_" device="01005" package3d_urn="urn:adsk.eagle:package:26133/1" value="330"/>
+<part name="R2" library="home" deviceset="R-US_" device="R0603" package3d_urn="urn:adsk.eagle:package:23555/2" value="330"/>
 <part name="C3" library="home" deviceset="MUR-1220-CAP" device="" value="MUR-1220-CAP"/>
+<part name="R3" library="home" deviceset="R-US_" device="R0603" package3d_urn="urn:adsk.eagle:package:23555/2" value="75"/>
 </parts>
 <sheets>
@@
 <attribute name="NAME" x="185.1914" y="54.9656" size="2.0828" layer="95" ratio="10" rot="SR180"/>
 </instance>
+<instance part="R3" gate="G$1" x="160.02" y="55.88" rot="R90"/>
 </instances>
 <busses>
@@
 <pinref part="JP4" gate="G$1" pin="1"/>
 <wire x1="200.66" y1="40.64" x2="200.66" y2="66.04" width="0.1524" layer="91"/>
-<pinref part="POWER" gate="A" pin="33"/>
-<wire x1="160.02" y1="45.72" x2="160.02" y2="66.04" width="0.1524" layer="91"/>
 <junction x="160.02" y="66.04"/>
 <label x="162.56" y="63.5" size="1.778" layer="95"/>
+<pinref part="R3" gate="G$1" pin="2"/>
+<wire x1="160.02" y1="60.96" x2="160.02" y2="66.04" width="0.1524" layer="91"/>
 </segment>
 <segment>
@@
 </segment>
 </net>
-<net name="N$62" class="0">
+<net name="GPA0" class="0">
 <segment>
 <pinref part="U1" gate="A" pin="I1"/>
@@
 </segment>
 </net>
-<net name="N$63" class="0">
+<net name="GPB0" class="0">
 <segment>
 <pinref part="U3" gate="G$1" pin="GPB0"/>
@@
 </segment>
 </net>
-<net name="N$64" class="0">
+<net name="GPA1" class="0">
 <segment>
 <pinref part="U1" gate="A" pin="I3"/>
@@
 </segment>
 </net>
-<net name="N$65" class="0">
+<net name="GPA2" class="0">
 <segment>
 <pinref part="U1" gate="A" pin="I5"/>
@@
 </segment>
 </net>
-<net name="N$66" class="0">
+<net name="GPB2" class="0">
 <segment>
 <wire x1="58.42" y1="92.71" x2="58.42" y2="118.11" width="0.1524" layer="91"/>
@@
 </segment>
 </net>
-<net name="N$67" class="0">
+<net name="GPB1" class="0">
 <segment>
 <wire x1="60.96" y1="90.17" x2="60.96" y2="115.57" width="0.1524" layer="91"/>
@@
 </segment>
 </net>
-<net name="N$74" class="0">
+<net name="GPA7" class="0">
 <segment>
 <pinref part="U3" gate="G$1" pin="GPA7"/>
@@
 </segment>
 </net>
-<net name="N$75" class="0">
+<net name="GPB5" class="0">
 <segment>
 <pinref part="U3" gate="G$1" pin="GPB5"/>
@@
 </segment>
 </net>
-<net name="N$76" class="0">
+<net name="GPB6" class="0">
 <segment>
 <pinref part="U3" gate="G$1" pin="GPB6"/>
@@
 </segment>
 </net>
-<net name="N$77" class="0">
+<net name="GPB7" class="0">
 <segment>
 <pinref part="U3" gate="G$1" pin="GPB7"/>
@@
 </segment>
 </net>
-<net name="N$68" class="0">
+<net name="GPA3" class="0">
 <segment>
 <pinref part="U2" gate="A" pin="I1"/>
@@
 </segment>
 </net>
-<net name="N$69" class="0">
+<net name="GPB3" class="0">
 <segment>
 <pinref part="U3" gate="G$1" pin="GPB3"/>
@@
 </segment>
 </net>
-<net name="N$70" class="0">
+<net name="GPA4" class="0">
 <segment>
 <pinref part="U3" gate="G$1" pin="GPA4"/>
@@
 </segment>
 </net>
-<net name="N$71" class="0">
+<net name="GPB4" class="0">
 <segment>
 <pinref part="U2" gate="A" pin="I4"/>
@@
 </segment>
 </net>
-<net name="N$80" class="0">
+<net name="GPA5" class="0">
 <segment>
 <pinref part="U3" gate="G$1" pin="GPA5"/>
@@
 </segment>
 </net>
-<net name="N$81" class="0">
+<net name="GPA6" class="0">
 <segment>
 <pinref part="U3" gate="G$1" pin="GPA6"/>
@@
 </segment>
 </net>
+<net name="N$2" class="0">
+<segment>
+<pinref part="R3" gate="G$1" pin="1"/>
+<pinref part="POWER" gate="A" pin="33"/>
+<wire x1="160.02" y1="45.72" x2="160.02" y2="50.8" width="0.1524" layer="91"/>
+</segment>
+</net>
